Commit message: Create separate file for T265 description

File: src/robot_description/urdf/robot_description.urdf.xacro (robot description, xacro)
@@ -79,17 +79,7 @@
     <origin xyz="${offset_435_x} ${body_length/2 + d435_offset_y + mount_offset_435} ${body_height/2 - 0.0254}" rpy="0 0 ${pi/2}"/>
   </xacro:sensor_d435>
-  <!--Create the 265 macro-->
-  <xacro:macro name="sensor_t265" params="parent">
-    <link name="sensor_t265">
-      <visual>
-        <geometry>
-          <box size="0.10795 0.0127 0.0254"/>
-        </geometry>
-      </visual>
-    </link>
-    <link name="fisheye_1"/>
-    <link name="fisheye_2"/>
-    <link name="imu"/>
-    <link name="t265_pose"/>
-  </xacro:macro>
+  <xacro:include filename="$(find realsense2_description)/urdf/_t265.urdf.xacro"/>
+  <xacro:sensor_t265 parent="body">
+    <origin xyz="0.0 ${body_length/2 + 0.0508} 0.0" rpy="0.0 0.0 0.0"/>
+  </xacro:sensor_t265>
 </robot>

Commit message: .

File: src/robot_description/urdf/robot_description.urdf.xacro (robot description, xacro)
@@ -31,8 +31,8 @@
     <xacro:robot_wheel prefix="${prefix}" number="${number}"/>
     <joint name="${prefix}_wheel_${number}_joint" type="fixed">
-      <parent link="base_link"/>
+      <parent link="body"/>
       <child link="${prefix}_wheel_${number}"/>
-      <!--axis xyz="0.0 1.0 0.0"/-->
-      <origin xyz="${((robot_width/2) - (wheel_width/2))*reflect} ${(wheelbase/2 - wheel_radius)*(number-2)*-1} ${wheel_radius}"/>
+      <!--axis xyz="0.0 1.0 0.0" rpy="0 0 0"/-->
+      <origin xyz="${((robot_width/2) - (wheel_width/2))*reflect} ${(wheelbase/2 - wheel_radius)*(number-2)*-1} ${wheel_radius - (robot_height - body_height/2)}"/>
     </joint>
   </xacro:macro>
