Commit message: Updated to work on running robot, not just simulation

File: src/realsense-ros-2.2.17/realsense2_description/urdf/_t265.urdf.xacro (robot description, xacro)
@@ -33,5 +33,5 @@
     <link name="fisheye2"/>
     <!--link name="imu"/-->
-    <link name="t265_pose"/>
+    <link name="t265_pose_frame"/>
     <joint name="fisheye1_joint" type="fixed">
       <parent link="sensor_t265"/>
@@ -46,5 +46,5 @@
     <joint name="pose_joint" type="fixed">
       <parent link="sensor_t265"/>
-      <child link="t265_pose"/>
+      <child link="t265_pose_frame"/>
       <origin xyz="${pose_offset_x} ${sensor_offset_y} 0.0" rpy="${pi/2} 0.0 0.0"/>
     </joint>

Commit message: Redifine the coordinate system to make the 265 the parent frame for odom transforms

File: src/realsense-ros-2.2.17/realsense2_description/urdf/_t265.urdf.xacro (robot description, xacro)
@@ -12,5 +12,5 @@
   <xacro:property name="zero_depth_to_glass" value="4.2e-3"/>
   <!--Create the 265 macro-->
-  <xacro:macro name="sensor_t265" params="parent *origin">
+  <xacro:macro name="sensor_t265" params="child *origin">
     <xacro:property name="t265_width" value="0.10795" />
     <xacro:property name="t265_depth" value="0.0127" />
@@ -19,5 +19,5 @@
     <xacro:property name="fisheye2_offset_x" value="${t265_width/2 - (t265_width - 0.0762)}" />
     <xacro:property name="pose_offset_x" value="${(fisheye1_offset_x+fisheye2_offset_x)/2}" />
-    <xacro:property name="sensor_offset_y" value="${t265_depth - glass_to_front - zero_depth_to_glass}" />
+    <xacro:property name="sensor_offset_y" value="${t265_depth/2 - glass_to_front - zero_depth_to_glass}" />
     <link name="sensor_t265">
       <visual>
@@ -33,5 +33,5 @@
     <link name="fisheye2"/>
     <!--link name="imu"/-->
-    <link name="t265_pose_frame"/>
+    <link name="t265_pose"/>
     <joint name="fisheye1_joint" type="fixed">
       <parent link="sensor_t265"/>
@@ -45,12 +45,12 @@
     </joint>
     <joint name="pose_joint" type="fixed">
-      <parent link="sensor_t265"/>
-      <child link="t265_pose_frame"/>
-      <origin xyz="${pose_offset_x} ${sensor_offset_y} 0.0" rpy="${pi/2} 0.0 0.0"/>
+      <parent link="t265_pose"/>
+      <child link="sensor_t265"/>
+      <origin xyz="${-pose_offset_x} 0.0 ${sensor_offset_y}" rpy="${-pi/2} 0.0 0.0"/>
     </joint>
     <joint name="t265_joint" type="fixed">
       <xacro:insert_block name="origin" />
-      <parent link="${parent}"/>
-      <child link="sensor_t265"/>
+      <parent link="sensor_t265"/>
+      <child link="${child}"/>
     </joint>
   </xacro:macro>

File: src/robot_controller/urdf/robot_description.urdf.xacro (robot description, xacro)
@@ -69,7 +69,7 @@
   </link>
   <joint name="body_link" type="fixed">
-    <parent link="base_link"/>
-    <child link="body"/>
-    <origin xyz="0 0 ${robot_height - body_height/2}"/>
+    <parent link="body"/>
+    <child link="base_link"/>
+    <origin xyz="0 0 ${-(robot_height - body_height/2)}"/>
   </joint>
   <!--Create all the wheels and define all the wheel joints-->
@@ -97,6 +97,9 @@
   </xacro:sensor_d435>
   <xacro:include filename="$(find realsense2_description)/urdf/_t265.urdf.xacro"/>
-  <xacro:sensor_t265 parent="body">
-    <origin xyz="0.0 ${body_length/2 + 0.0508} 0.0" rpy="0.0 0.0 0.0"/>
+  <xacro:property name="t265_width" value="0.10795" />
+  <xacro:property name="t265_depth" value="0.0127" />
+  <xacro:property name="t265_height" value="0.0254" />
+  <xacro:sensor_t265 child="body">
+    <origin xyz="${body_width/2 - (t265_width/2 + 0.1571625)} ${-(body_length/2 + t265_depth/2 + 0.0238125)} 0.0" rpy="0.0 0.0 0.0"/>
   </xacro:sensor_t265>
 </robot>

Commit message: Updated transforms to transform reference frames properly

File: src/realsense-ros-2.2.17/realsense2_description/urdf/_t265.urdf.xacro (robot description, xacro)
@@ -33,5 +33,5 @@
     <link name="fisheye2"/>
     <!--link name="imu"/-->
-    <link name="t265_pose"/>
+    <link name="t265_pose_link"/>
     <joint name="fisheye1_joint" type="fixed">
       <parent link="sensor_t265"/>
@@ -45,5 +45,5 @@
     </joint>
     <joint name="pose_joint" type="fixed">
-      <parent link="t265_pose"/>
+      <parent link="t265_pose_link"/>
       <child link="sensor_t265"/>
       <origin xyz="${-pose_offset_x} 0.0 ${sensor_offset_y}" rpy="${-pi/2} 0.0 0.0"/>

Commit message: Fixed incorrect rotation value between t265 and pose frame. librealsense uses VR coordinate frame (which is how the camera is documented). But the ROS wrapper uses ROS standards

File: src/realsense-ros-2.2.17/realsense2_description/urdf/_t265.urdf.xacro (robot description, xacro)
@@ -47,5 +47,5 @@
       <parent link="t265_pose_link"/>
       <child link="sensor_t265"/>
-      <origin xyz="${-pose_offset_x} 0.0 ${sensor_offset_y}" rpy="${-pi/2} 0.0 0.0"/>
+      <origin xyz="${-pose_offset_x} 0.0 ${sensor_offset_y}" rpy="0.0 0.0 ${-pi/2}"/>
     </joint>
     <joint name="t265_joint" type="fixed">

Commit message: Integrate the roboclaw with the cameras

File: src/realsense-ros-2.2.17/realsense2_description/urdf/_t265.urdf.xacro (robot description, xacro)
@@ -47,5 +47,5 @@
       <parent link="t265_pose_link"/>
       <child link="sensor_t265"/>
-      <origin xyz="${-pose_offset_x} 0.0 ${sensor_offset_y}" rpy="0.0 0.0 ${-pi/2}"/>
+      <origin xyz="0.0 ${pose_offset_x} 0.0" rpy="0.0 0.0 ${-pi/2}"/>
     </joint>
     <joint name="t265_joint" type="fixed">

File: src/robot_controller/urdf/robot_description.urdf.xacro (robot description, xacro)
@@ -49,4 +49,5 @@
   </xacro:macro>
   <link name="base_link"/>
+  <link name="wheel_odom_link"/>
   <link name="body">
     <visual name="body_visual">
@@ -68,8 +69,13 @@
     </collision>
   </link>
-  <joint name="body_link" type="fixed">
+  <joint name="body_joint" type="fixed">
     <parent link="body"/>
     <child link="base_link"/>
     <origin xyz="0 0 ${-(robot_height - body_height/2)}"/>
+  </joint>
+  <joint name="wheel_odom_joint" type="fixed">
+    <parent link="base_link"/>
+    <child link="wheel_odom_link"/>
+    <origin xyz="0.0 0.0 ${wheel_radius}" rpy="0.0 0.0 ${pi/2}"/>
   </joint>
   <!--Create all the wheels and define all the wheel joints-->
@@ -102,5 +108,5 @@
   <xacro:property name="t265_height" value="0.0254" />
   <xacro:sensor_t265 child="body">
-    <origin xyz="${body_width/2 - (t265_width/2 + 0.1571625)} ${-(body_length/2 + t265_depth/2 + 0.0238125)} 0.0" rpy="0.0 0.0 0.0"/>
+    <origin xyz="${body_width/2 - (t265_width/2 + 0.1571625)} ${-(body_length/2 + t265_depth/2 + 0.0238125)} ${-body_height/2 + t265_height/2 + 0.0301625}" rpy="0.0 0.0 0.0"/>
   </xacro:sensor_t265>
 </robot>

Commit message: Swap coordinate frame so that x is forward to match ros conventions

File: src/realsense-ros-2.2.17/realsense2_description/urdf/_t265.urdf.xacro (robot description, xacro)
@@ -16,12 +16,12 @@
     <xacro:property name="t265_depth" value="0.0127" />
     <xacro:property name="t265_height" value="0.0254" />
-    <xacro:property name="fisheye1_offset_x" value="${0.0127 - t265_width/2}" />
-    <xacro:property name="fisheye2_offset_x" value="${t265_width/2 - (t265_width - 0.0762)}" />
-    <xacro:property name="pose_offset_x" value="${(fisheye1_offset_x+fisheye2_offset_x)/2}" />
-    <xacro:property name="sensor_offset_y" value="${t265_depth/2 - glass_to_front - zero_depth_to_glass}" />
+    <xacro:property name="fisheye1_offset_y" value="${t265_width/2 - 0.0127}" />
+    <xacro:property name="fisheye2_offset_y" value="${t265_width/2 - 0.0762}" />
+    <xacro:property name="pose_offset_y" value="${(fisheye1_offset_y+fisheye2_offset_y)/2}" />
+    <xacro:property name="sensor_offset_x" value="${t265_depth/2 - glass_to_front - zero_depth_to_glass}" />
     <link name="sensor_t265">
       <visual>
         <geometry>
-          <box size="${t265_width} ${t265_depth} ${t265_height}"/>
+          <box size="${t265_depth} ${t265_width} ${t265_height}"/>
         </geometry>
         <material name="grey">
@@ -37,15 +37,15 @@
       <parent link="sensor_t265"/>
       <child link="fisheye1"/>
-      <origin xyz="${fisheye1_offset_x} ${sensor_offset_y} 0.0" rpy="${-pi/2} 0.0 0.0"/>
+      <origin xyz="${sensor_offset_x} ${fisheye1_offset_y} 0.0" rpy="${-pi/2} 0.0 ${-pi/2}"/>
     </joint>
     <joint name="fisheye2_joint" type="fixed">
       <parent link="sensor_t265"/>
       <child link="fisheye2"/>
-      <origin xyz="${fisheye2_offset_x} ${sensor_offset_y} 0.0" rpy="${-pi/2} 0.0 0.0"/>
+      <origin xyz="${sensor_offset_x} ${fisheye2_offset_y} 0.0" rpy="${-pi/2} 0.0 ${-pi/2}"/>
     </joint>
     <joint name="pose_joint" type="fixed">
       <parent link="t265_pose_link"/>
       <child link="sensor_t265"/>
-      <origin xyz="0.0 ${pose_offset_x} 0.0" rpy="0.0 0.0 ${-pi/2}"/>
+      <origin xyz="0.0 ${-pose_offset_y} 0.0" rpy="0.0 0.0 0.0"/>
     </joint>
     <joint name="t265_joint" type="fixed">

File: src/robot_controller/urdf/robot_description.urdf.xacro (robot description, xacro)
@@ -14,5 +14,5 @@
     <link name="${prefix}_wheel_${number}">
       <inertial>
-        <origin rpy="0.0 ${pi/2} 0.0"/>
+        <origin rpy="${pi/2} 0.0 0.0"/>
         <mass value="1"/>
         <cylinder_inertia m="1" r="${wheel_radius}" h="${wheel_width}"/>
@@ -23,5 +23,5 @@
       </inertial>
       <visual name="${prefix}_wheel_${number}_visual">
-        <origin rpy="0.0 ${pi/2} 0.0"/>
+        <origin rpy="${pi/2} 0.0 0.0"/>
         <geometry>
           <cylinder radius="${wheel_radius}" length="${wheel_width}"/>
@@ -32,5 +32,5 @@
       </visual>
       <collision>
-        <origin rpy="0.0 ${pi/2} 0.0"/>
+        <origin rpy="${pi/2} 0.0 0.0"/>
         <geometry>
           <cylinder radius="${wheel_radius}" length="${wheel_width}"/>
@@ -44,6 +44,6 @@
       <parent link="body"/>
       <child link="${prefix}_wheel_${number}"/>
-      <axis xyz="1.0 0.0 0.0" rpy="0 0 0"/>
-      <origin xyz="${((robot_width/2) - (wheel_width/2))*reflect} ${(wheelbase/2 - wheel_radius)*(number-2)*-1} ${wheel_radius - (robot_height - body_height/2)}"/>
+      <axis xyz="0.0 1.0 0.0" rpy="0 0 0"/>
+      <origin xyz="${(wheelbase/2 - wheel_radius)*(number-2)*-1} ${((robot_width/2) - (wheel_width/2))*reflect} ${wheel_radius - (robot_height - body_height/2)}"/>
     </joint>
   </xacro:macro>
@@ -53,5 +53,5 @@
     <visual name="body_visual">
       <geometry>
-        <box size="${body_width} ${body_length} ${body_height}"/>
+        <box size="${body_length} ${body_width} ${body_height}"/>
       </geometry>
     </visual>
@@ -65,5 +65,5 @@
     <collision>
       <geometry>
-        <box size="${body_width} ${body_length} ${body_height}"/>
+        <box size="${body_length} ${body_width} ${body_height}"/>
       </geometry>
     </collision>
@@ -77,13 +77,13 @@
     <parent link="base_link"/>
     <child link="wheel_odom_link"/>
-    <origin xyz="0.0 0.0 ${wheel_radius}" rpy="0.0 0.0 ${pi/2}"/>
+    <origin xyz="0.0 0.0 ${wheel_radius}" rpy="0.0 0.0 0.0"/>
   </joint>
   <!--Create all the wheels and define all the wheel joints-->
-  <xacro:wheel_joint prefix="left" reflect="-1" number="1"/>
-  <xacro:wheel_joint prefix="left" reflect="-1" number="2"/>
-  <xacro:wheel_joint prefix="left" reflect="-1" number="3"/>
-  <xacro:wheel_joint prefix="right" reflect="1" number="1"/>
-  <xacro:wheel_joint prefix="right" reflect="1" number="2"/>
-  <xacro:wheel_joint prefix="right" reflect="1" number="3"/>
+  <xacro:wheel_joint prefix="left" reflect="1" number="1"/>
+  <xacro:wheel_joint prefix="left" reflect="1" number="2"/>
+  <xacro:wheel_joint prefix="left" reflect="1" number="3"/>
+  <xacro:wheel_joint prefix="right" reflect="-1" number="1"/>
+  <xacro:wheel_joint prefix="right" reflect="-1" number="2"/>
+  <xacro:wheel_joint prefix="right" reflect="-1" number="3"/>
   <!--Import the 435 model-->
   <xacro:include filename="$(find realsense2_description)/urdf/_d435.urdf.xacro"/>
@@ -96,9 +96,9 @@
   <xacro:property name="zero_depth_to_glass" value="4.2e-3"/>
   <!-- convenience precomputation to avoid clutter-->
-  <xacro:property name="d435_offset_y" value="${d435_cam_mount_from_center_offset-glass_to_front-zero_depth_to_glass}"/>
-  <xacro:property name="offset_435_x" value="${body_width/2 - 0.2032}"/>
+  <xacro:property name="d435_offset_x" value="${d435_cam_mount_from_center_offset-glass_to_front-zero_depth_to_glass}"/>
+  <xacro:property name="offset_435_y" value="${body_width/2 - 0.2032}"/>
   <xacro:property name="mount_offset_435" value="0.0111125"/>
   <xacro:sensor_d435 parent="body">
-    <origin xyz="${offset_435_x} ${body_length/2 + d435_offset_y + mount_offset_435} ${body_height/2 - 0.0254}" rpy="0 0 ${pi/2}"/>
+    <origin xyz="${body_length/2 + d435_offset_x + mount_offset_435} ${offset_435_y} ${body_height/2 - 0.0254}" rpy="0 0 0"/>
   </xacro:sensor_d435>
   <!--Import the 265 model-->
@@ -108,5 +108,5 @@
   <xacro:property name="t265_height" value="0.0254" />
   <xacro:sensor_t265 child="body">
-    <origin xyz="${body_width/2 - (t265_width/2 + 0.1571625)} ${-(body_length/2 + t265_depth/2 + 0.0238125)} ${-body_height/2 + t265_height/2 + 0.0301625}" rpy="0.0 0.0 0.0"/>
+    <origin xyz="${-(body_length/2 + t265_depth/2 + 0.0238125)} ${-body_width/2 + 0.1571625 + t265_width/2} ${-body_height/2 + t265_height/2 + 0.0301625}" rpy="0.0 0.0 0.0"/>
   </xacro:sensor_t265>
 </robot>
