Commit message: Created running gazebo model (moving simulation untested)

File: src/robot_controller/urdf/robot_description.urdf.xacro (robot description, xacro)
@@ -1,4 +1,5 @@
 <?xml version="1.0"?>
 <robot name="robot_base" xmlns:xacro="http://ros.org/wiki/xacro">
+  <xacro:include filename="$(find robot_controller)/urdf/mybot.gazebo"/>
   <xacro:property name="robot_width" value="0.57375" />
   <xacro:property name="robot_length" value="0.5032"/>
@@ -14,8 +15,12 @@
       <inertial>
         <origin rpy="0.0 ${pi/2} 0.0"/>
-        <mass value="0.0"/>
-        <inertia ixx="0.0" ixy="0.0" ixz="0.0" iyy="0.0" iyz="0.0" izz="0.0"/>
+        <mass value="5"/>
+        <cylinder_inertia m="5" r="${wheel_radius}" h="${wheel_width}"/>
+        <inertia
+            ixx="1.0" ixy="0.0" ixz="0.0"
+            iyy="1.0" iyz="0.0"
+            izz="1.0"/>
       </inertial>
-      <visual name="wheel">
+      <visual name="${prefix}_wheel_${number}_visual">
         <origin rpy="0.0 ${pi/2} 0.0"/>
         <geometry>
@@ -26,28 +31,40 @@
         </material>
       </visual>
+      <collision>
+        <origin rpy="0.0 ${pi/2} 0.0"/>
+        <geometry>
+          <cylinder radius="${wheel_radius}" length="${wheel_width}"/>
+        </geometry>
+      </collision>
     </link>
   </xacro:macro>
   <xacro:macro name="wheel_joint" params="prefix reflect number">
     <xacro:robot_wheel prefix="${prefix}" number="${number}"/>
-    <joint name="${prefix}_wheel_${number}_joint" type="fixed">
+    <joint name="${prefix}_wheel_${number}_joint" type="continuous">
       <parent link="body"/>
       <child link="${prefix}_wheel_${number}"/>
-      <!--axis xyz="0.0 1.0 0.0" rpy="0 0 0"/-->
+      <axis xyz="1.0 0.0 0.0" rpy="0 0 0"/>
       <origin xyz="${((robot_width/2) - (wheel_width/2))*reflect} ${(wheelbase/2 - wheel_radius)*(number-2)*-1} ${wheel_radius - (robot_height - body_height/2)}"/>
     </joint>
   </xacro:macro>
-  <link name="base_link">
-    <collision>
-      <geometry>
-        <box size="${robot_width} ${robot_length} ${robot_height}"/>
-      </geometry>
-    </collision>
-  </link>
+  <link name="base_link"/>
   <link name="body">
-    <visual>
+    <visual name="body_visual">
       <geometry>
         <box size="${body_width} ${body_length} ${body_height}"/>
       </geometry>
     </visual>
+    <inertial>
+      <mass value="10.0"/>
+      <inertia
+            ixx="0.5" ixy="0.0" ixz="0.0"
+            iyy="1.0" iyz="0.0"
+            izz="0.1"/>
+    </inertial>
+    <collision>
+      <geometry>
+        <box size="${body_width} ${body_length} ${body_height}"/>
+      </geometry>
+    </collision>
   </link>
   <joint name="body_link" type="fixed">

Commit message: Modify simulation settings for smoother driving

File: src/robot_controller/urdf/robot_description.urdf.xacro (robot description, xacro)
@@ -15,10 +15,10 @@
       <inertial>
         <origin rpy="0.0 ${pi/2} 0.0"/>
-        <mass value="5"/>
-        <cylinder_inertia m="5" r="${wheel_radius}" h="${wheel_width}"/>
+        <mass value="1"/>
+        <cylinder_inertia m="1" r="${wheel_radius}" h="${wheel_width}"/>
         <inertia
-            ixx="1.0" ixy="0.0" ixz="0.0"
-            iyy="1.0" iyz="0.0"
-            izz="1.0"/>
+            ixx="0.1" ixy="0.0" ixz="0.0"
+            iyy="0.1" iyz="0.0"
+            izz="0.1"/>
       </inertial>
       <visual name="${prefix}_wheel_${number}_visual">
@@ -56,5 +56,5 @@
     </visual>
     <inertial>
-      <mass value="10.0"/>
+      <mass value="1.0"/>
       <inertia
             ixx="0.5" ixy="0.0" ixz="0.0"
@@ -96,4 +96,5 @@
     <origin xyz="${offset_435_x} ${body_length/2 + d435_offset_y + mount_offset_435} ${body_height/2 - 0.0254}" rpy="0 0 ${pi/2}"/>
   </xacro:sensor_d435>
+  <!--Import the 265 model-->
   <xacro:include filename="$(find realsense2_description)/urdf/_t265.urdf.xacro"/>
   <xacro:sensor_t265 parent="body">

Commit message: restructure simulation environment

File: src/robot_controller/urdf/robot_description.urdf.xacro (robot description, xacro)
@@ -1,5 +1,5 @@
 <?xml version="1.0"?>
 <robot name="robot_base" xmlns:xacro="http://ros.org/wiki/xacro">
-  <xacro:include filename="$(find robot_controller)/urdf/mybot.gazebo"/>
+  <xacro:include filename="$(find robot_controller)/xacro/inertia_calc.xacro"/>
   <xacro:property name="robot_width" value="0.57375" />
   <xacro:property name="robot_length" value="0.5032"/>
@@ -8,17 +8,15 @@
   <xacro:property name="body_length" value="0.5032"/>
   <xacro:property name="body_height" value="0.08255"/>
+  <xacro:property name="body_mass" value="11"/>
   <xacro:property name="wheel_radius" value="0.066675"/>
   <xacro:property name="wheel_width" value="0.05715"/>
   <xacro:property name="wheelbase" value="0.4826"/>
+  <xacro:property name="wheel_mass" value="0.45"/>
   <xacro:macro name="robot_wheel" params="prefix number">
     <link name="${prefix}_wheel_${number}">
       <inertial>
         <origin rpy="${pi/2} 0.0 0.0"/>
-        <mass value="1"/>
-        <cylinder_inertia m="1" r="${wheel_radius}" h="${wheel_width}"/>
-        <inertia
-            ixx="0.1" ixy="0.0" ixz="0.0"
-            iyy="0.1" iyz="0.0"
-            izz="0.1"/>
+        <mass value="${wheel_mass}"/>
+        <xacro:cylinder_inertia m="${wheel_mass}" r="${wheel_radius}" h="${wheel_width}"/>
       </inertial>
       <visual name="${prefix}_wheel_${number}_visual">
@@ -36,4 +34,22 @@
           <cylinder radius="${wheel_radius}" length="${wheel_width}"/>
         </geometry>
+        <surface>
+          <friction>
+            <ode>
+              <mu1>1.0</mu1>
+              <mu2>1.0</mu2>
+              <slip1>0.0</slip1>
+              <slip2>0.0</slip2>
+            </ode>
+          </friction>
+          <contact>
+            <ode>
+              <kp>1000000.0</kp> <!-- kp and kd for rubber -->
+              <kd>100.0</kd>
+              <maxVel>1.0</maxVel>
+              <minDepth>0.00</minDepth>
+            </ode>
+          </contact>
+        </surface>
       </collision>
     </link>
@@ -57,9 +73,6 @@
     </visual>
     <inertial>
-      <mass value="1.0"/>
-      <inertia
-            ixx="0.5" ixy="0.0" ixz="0.0"
-            iyy="1.0" iyz="0.0"
-            izz="0.1"/>
+      <mass value="${body_mass}"/>
+      <xacro:box_inertia m="${body_mass}" x="${body_length}" y="${body_width}" z="${body_height}"/>
     </inertial>
     <collision>
